Commit message: feat: Add head link and joint to the legged robot URDF

File: src/robot/urdf/legged_robot.urdf (robot description, URDF)
Before this commit: robot legged_robot, 25 links, 24 joints
Links:
- added link head, mass 0.1; collision box size=0.2 0.15 0.1; visual box size=0.2 0.15 0.1
Joints:
- added joint body_to_head: type fixed, parent base_link, child head, origin xyz=0.5 0 0.2 rpy=0 0 0

Commit message: fix: Correct joint axis direction for leg joints in URDF

File: src/robot/urdf/legged_robot.urdf (robot description, URDF)
Before this commit: robot legged_robot, 26 links, 25 joints
Joints:
- joint joint_0: axis 0 1 0 -> 0 -1 0
- joint joint_12: axis 0 1 0 -> 0 -1 0
- joint joint_15: axis 0 1 0 -> 0 -1 0
- joint joint_3: axis 0 1 0 -> 0 -1 0
- joint joint_6: axis 0 1 0 -> 0 -1 0
- joint joint_9: axis 0 1 0 -> 0 -1 0

Commit message: fix: Invert joint axis direction for left side legs in URDF generation

File: src/robot/urdf/legged_robot.urdf (robot description, URDF)
Before this commit: robot legged_robot, 26 links, 25 joints
Joints:
- joint joint_10: axis 1 0 0 -> -1 0 0
- joint joint_11: axis 1 0 0 -> -1 0 0
- joint joint_13: axis 1 0 0 -> -1 0 0
- joint joint_14: axis 1 0 0 -> -1 0 0
- joint joint_16: axis 1 0 0 -> -1 0 0
- joint joint_17: axis 1 0 0 -> -1 0 0

Commit message: fix: Correct joint axis directions for leg joints in URDF and locomotion logic

File: src/robot/urdf/legged_robot.urdf (robot description, URDF)
Before this commit: robot legged_robot, 26 links, 25 joints
Joints:
- joint joint_0: axis 0 -1 0 -> 0 1 0
- joint joint_1: axis 1 0 0 -> -1 0 0
- joint joint_12: axis 0 -1 0 -> 0 1 0
- joint joint_15: axis 0 -1 0 -> 0 1 0
- joint joint_2: axis 1 0 0 -> -1 0 0
- joint joint_3: axis 0 -1 0 -> 0 1 0
- joint joint_4: axis 1 0 0 -> -1 0 0
- joint joint_5: axis 1 0 0 -> -1 0 0
- joint joint_6: axis 0 -1 0 -> 0 1 0
- joint joint_7: axis 1 0 0 -> -1 0 0
- joint joint_8: axis 1 0 0 -> -1 0 0
- joint joint_9: axis 0 -1 0 -> 0 1 0
